File: coilgun_stage_v1/coilgun_stage.sch (KiCad schematic (older format))
At the start: 16 parts, among them J1 Conn_01x05_Female, J2 Conn_01x05_Female, Q1 MMBT5551L, Q2 LTR-4206E

Commit message: Get rid of the useless optocoupler
Parts:
- R1, R2, R3, R4: footprint Resistor_SMD:R_0603_1608Metric -> Resistor_SMD:R_0603_1608Metric_Pad0.98x0.95mm_HandSolder
Changed lines of the file:
@@
 F 0 "R2" H 3409 1346 50  0000 L CNN
 F 1 "0" H 3409 1255 50  0000 L CNN
-F 2 "Resistor_SMD:R_0603_1608Metric" H 3350 1300 50  0001 C CNN
+F 2 "Resistor_SMD:R_0603_1608Metric_Pad0.98x0.95mm_HandSolder" H 3350 1300 50  0001 C CNN
 F 3 "~" H 3350 1300 50  0001 C CNN
 	1    3350 1300
@@
 F 0 "R1" V 2754 1600 50  0000 C CNN
 F 1 "5.6k" V 2845 1600 50  0000 C CNN
-F 2 "Resistor_SMD:R_0603_1608Metric" H 2950 1600 50  0001 C CNN
+F 2 "Resistor_SMD:R_0603_1608Metric_Pad0.98x0.95mm_HandSolder" H 2950 1600 50  0001 C CNN
 F 3 "~" H 2950 1600 50  0001 C CNN
 	1    2950 1600
@@
 F 0 "R3" H 5559 1946 50  0000 L CNN
 F 1 "100" H 5559 1855 50  0000 L CNN
-F 2 "Resistor_SMD:R_0603_1608Metric" H 5500 1900 50  0001 C CNN
+F 2 "Resistor_SMD:R_0603_1608Metric_Pad0.98x0.95mm_HandSolder" H 5500 1900 50  0001 C CNN
 F 3 "~" H 5500 1900 50  0001 C CNN
 	1    5500 1900
@@
 F 0 "R4" H 6309 1896 50  0000 L CNN
 F 1 "1k" H 6309 1805 50  0000 L CNN
-F 2 "Resistor_SMD:R_0603_1608Metric" H 6250 1850 50  0001 C CNN
+F 2 "Resistor_SMD:R_0603_1608Metric_Pad0.98x0.95mm_HandSolder" H 6250 1850 50  0001 C CNN
 F 3 "~" H 6250 1850 50  0001 C CNN
 	1    6250 1850
